Commit message: 对botyard hand进行了评估

File: assets/botyard_left/botyard_hand_left.urdf (robot description, URDF)
Before this commit: robot dexhand, 33 links, 32 joints
Joints:
- joint FAJ1: origin xyz=0 -0.0193 0.039 rpy=0 0 -1.5708 -> xyz=0 -0.0193 0.039 rpy=0 0 0; type revolute -> fixed
- joint FAJ3: type revolute -> fixed
- joint LFJ5: type revolute -> fixed
